Commit message: Update vlp16-imu.urdf

File: cartographer_key/cartographer_ros/urdf/vlp16-imu.urdf (robot description, URDF)
Before this commit: robot jackal, 3 links, 2 joints
Links:
- removed link imu_link
- added link kvh_link; visual box size=0.06 0.04 0.02
Joints:
- removed joint imu_to_base
- added joint kvh_to_base: type fixed, parent base_link, child kvh_link, origin xyz=0 0 0.24 rpy=0 0 0
- joint velodyne_to_base: origin xyz=0.0 0.0 0.5 rpy=0 0 0 -> xyz=0.0 0.0 0.48 rpy=0 0 0
